File: Thermocouple board Kicad/Thermocouple board/Thermocouple board.kicad_pcb (KiCad board)
At the start: 2 copper layers, 0 parts

Commit message: Add files via upload
Parts:
- added C1: .1 μF, cap:CAP_GRM155R61A106ME11_MUR_0402, F.Cu at (109.1, 49.4)
- added C10: .1 μF, cap:CAP_GRM155R61A106ME11_MUR_0402, F.Cu at (122.0, 68.1)
- added C11: .1 μF, cap:CAP_GRM155R61A106ME11_MUR_0402, F.Cu at (123.3, 68.2)
- added C13: 10 μF, cap:CAP_GRM155R61A106ME11_MUR_0402, F.Cu at (113.2, 50.8)
- added C14: 10 μF, cap:CAP_GRM155R61A106ME11_MUR_0402, F.Cu at (115.6, 49.3)
- added C15: 10 μF, cap:CAP_GRM155R61A106ME11_MUR_0402, F.Cu at (117.4, 49.5)
- added C16: .1 μF, cap:CAP_GRM155R61A106ME11_MUR_0402, F.Cu at (128.6, 54.6)
- added C17: .1 μF, cap:CAP_GRM155R61A106ME11_MUR_0402, F.Cu at (151.9, 120.2)
- added C18: .1 μF, cap:CAP_GRM155R61A106ME11_MUR_0402, F.Cu at (128.6, 58.2)
- added C19: .1 μF, cap:CAP_GRM155R61A106ME11_MUR_0402, F.Cu at (125.5, 68.2)
- added C2: 1 μF, cap:CAP_GRM155R61A106ME11_MUR_0402, F.Cu at (115.2, 63.0)
- added C20: .1 μF, cap:CAP_GRM155R61A106ME11_MUR_0402, F.Cu at (122.2, 108.1)
- added C21: .1 μF, cap:CAP_GRM155R61A106ME11_MUR_0402, F.Cu at (123.8, 102.7)
- added C22: .1 μF, cap:CAP_GRM155R61A106ME11_MUR_0402, F.Cu at (123.8, 89.9)
- added C23: .1 μF, cap:CAP_GRM155R61A106ME11_MUR_0402, F.Cu at (128.4, 74.8)
- added C24: .1 μF, cap:CAP_GRM155R61A106ME11_MUR_0402, F.Cu at (116.9, 107.9)
- added C26: .1 μF, cap:CAP_GRM155R61A106ME11_MUR_0402, F.Cu at (128.6, 53.2)
- added C3: 1 μF, cap:CAP_GRM155R61A106ME11_MUR_0402, F.Cu at (110.8, 58.2)
- added C4: .1 μF, cap:CAP_GRM155R61A106ME11_MUR_0402, F.Cu at (113.5, 68.0)
- added C5: .1 μF, cap:CAP_GRM155R61A106ME11_MUR_0402, F.Cu at (116.3, 68.0)
- added C6: .1 μF, cap:CAP_GRM155R61A106ME11_MUR_0402, F.Cu at (117.8, 68.0)
- added C7: .1 μF, cap:CAP_GRM155R61A106ME11_MUR_0402, F.Cu at (115.0, 68.0)
- added C8: .1 μF, cap:CAP_GRM155R61A106ME11_MUR_0402, F.Cu at (119.2, 68.0)
- added C9: .1 μF, cap:CAP_GRM155R61A106ME11_MUR_0402, F.Cu at (120.5, 68.1)
- added J1: Conn_01x06_Pin, Connector_PinHeader_2.54mm:PinHeader_1x06_P2.54mm_Vertical, F.Cu at (131.2, 41.0)
- added J2: Conn_01x02_Pin, Connector_PinHeader_2.54mm:PinHeader_1x02_P2.54mm_Vertical, F.Cu at (108.4, 41.0)
- added Q2: 2N3904, Package_TO_SOT_THT:TO-92_Inline, F.Cu at (125.5, 50.0)
- added Q3: 2N3904, Package_TO_SOT_THT:TO-92_Inline, F.Cu at (124.4, 63.2)
- added R1: 100 ohm, cap:RESC1607X60N, F.Cu at (102.5, 62.0)
- added R10: 100 ohm, cap:RESC1607X60N, F.Cu at (104.8, 93.8)
- added R11: 100 ohm, cap:RESC1607X60N, F.Cu at (104.2, 100.2)
- added R12: 100 ohm, cap:RESC1607X60N, F.Cu at (104.2, 103.8)
- added R13: 100 ohm, cap:RESC1607X60N, F.Cu at (104.8, 111.5)
- added R14: 100 ohm, cap:RESC1607X60N, F.Cu at (104.8, 115.3)
- added R15: 100 ohm, cap:RESC1607X60N, F.Cu at (103.1, 121.7)
- added R16: 100 ohm, cap:RESC1607X60N, F.Cu at (103.1, 125.4)
- added R17: 100 ohm, cap:RESC1607X60N, F.Cu at (111.0, 118.5)
- added R18: 100 ohm, cap:RESC1607X60N, F.Cu at (113.6, 118.5)
- added R19: 100 ohm, cap:RESC1607X60N, F.Cu at (121.9, 117.8)
- added R2: 100 ohm, cap:RESC1607X60N, F.Cu at (102.5, 65.5)
- added R20: 100 ohm, cap:RESC1607X60N, F.Cu at (125.3, 117.8)
- added R21: 100 ohm, cap:RESC1607X60N, F.Cu at (134.6, 117.3)
- added R22: 100 ohm, cap:RESC1607X60N, F.Cu at (134.6, 114.0)
- added R23: 100 ohm, cap:RESC1607X60N, F.Cu at (134.8, 107.4)
- added R24: 100 ohm, cap:RESC1607X60N, F.Cu at (135.0, 103.7)
- added R25: 100 ohm, cap:RESC1607X60N, F.Cu at (133.2, 98.6)
- added R26: 100 ohm, cap:RESC1607X60N, F.Cu at (133.7, 95.2)
- added R27: 100 ohm, cap:RESC1607X60N, F.Cu at (134.2, 89.5)
- added R28: 100 ohm, cap:RESC1607X60N, F.Cu at (134.0, 85.6)
- added R29: 100 ohm, cap:RESC1607X60N, F.Cu at (134.8, 80.3)
- added R3: 100 ohm, cap:RESC1607X60N, F.Cu at (104.5, 71.9)
- added R30: 100 ohm, cap:RESC1607X60N, F.Cu at (134.8, 76.8)
- added R31: 100 ohm, cap:RESC1607X60N, F.Cu at (133.6, 71.3)
- added R32: 100 ohm, cap:RESC1607X60N, F.Cu at (133.6, 67.8)
- added R33: 100 ohm, cap:RESC1607X60N, F.Cu at (134.8, 62.5)
- added R34: 100 ohm, cap:RESC1607X60N, F.Cu at (134.8, 58.8)
- added R35: 100 ohm, cap:RESC1607X60N, F.Cu at (135.2, 54.6)
- added R36: 100 ohm, cap:RESC1607X60N, F.Cu at (135.3, 51.0)
- added R4: 100 ohm, cap:RESC1607X60N, F.Cu at (104.4, 75.5)
- added R5: 100 ohm, cap:RESC1607X60N, F.Cu at (105.0, 81.5)
- added R6: 100 ohm, cap:RESC1607X60N, F.Cu at (104.5, 85.1)
- added R7: 100 ohm, cap:RESC1607X60N, F.Cu at (102.5, 51.5)
- added R8: 100 ohm, cap:RESC1607X60N, F.Cu at (102.5, 55.0)
- added R9: 100 ohm, cap:RESC1607X60N, F.Cu at (104.8, 90.3)
- added U1: LTC2984CLX-PBF, LTC2984:LQFP-48_LX_LIT, F.Cu at (117.8, 55.9)
- added X1: ~, Socket:TERMBLOCK_1X2-3.5MM, F.Cu at (97.0, 53.2)
- added X10: ~, Socket:TERMBLOCK_1X2-3.5MM, F.Cu at (123.5, 124.3)
- added X11: ~, Socket:TERMBLOCK_1X2-3.5MM, F.Cu at (141.3, 115.5)
- added X12: ~, Socket:TERMBLOCK_1X2-3.5MM, F.Cu at (141.2, 105.6)
- added X13: ~, Socket:TERMBLOCK_1X2-3.5MM, F.Cu at (141.1, 97.0)
- added X14: ~, Socket:TERMBLOCK_1X2-3.5MM, F.Cu at (140.9, 87.8)
- added X15: ~, Socket:TERMBLOCK_1X2-3.5MM, F.Cu at (140.8, 78.5)
- added X16: ~, Socket:TERMBLOCK_1X2-3.5MM, F.Cu at (141.1, 69.5)
- added X17: ~, Socket:TERMBLOCK_1X2-3.5MM, F.Cu at (141.1, 60.8)
- added X18: ~, Socket:TERMBLOCK_1X2-3.5MM, F.Cu at (141.1, 52.7)
- added X2: ~, Socket:TERMBLOCK_1X2-3.5MM, F.Cu at (97.0, 63.7)
- added X3: ~, Socket:TERMBLOCK_1X2-3.5MM, F.Cu at (97.0, 73.7)
- added X4: ~, Socket:TERMBLOCK_1X2-3.5MM, F.Cu at (97.0, 83.2)
- added X5: ~, Socket:TERMBLOCK_1X2-3.5MM, F.Cu at (96.9, 92.1)
- added X6: ~, Socket:TERMBLOCK_1X2-3.5MM, F.Cu at (97.2, 102.1)
- added X7: ~, Socket:TERMBLOCK_1X2-3.5MM, F.Cu at (97.1, 113.3)
- added X8: ~, Socket:TERMBLOCK_1X2-3.5MM, F.Cu at (97.0, 123.6)
- added X9: ~, Socket:TERMBLOCK_1X2-3.5MM, F.Cu at (112.2, 124.3)
Routing:
- net +3.3V: track 0.00 -> 33.6 mm
- net GND: track 0.00 -> 19.6 mm, vias 0 -> 15
- net Net-(U1-VREFOUT): track 0.00 -> 4.80 mm
- net Net-(U1-Q1): track 0.00 -> 3.12 mm
- net Net-(U1-Q2): track 0.00 -> 2.62 mm
- net Net-(U1-VREF_BYP): track 0.00 -> 2.18 mm
- net Net-(U1-Q3): track 0.00 -> 1.99 mm
- net Net-(U1-LDO): track 0.00 -> 1.66 mm
- net Net-(J1-Pin_1): track 0.00 -> 0.60 mm
- added copper zone on B.Cu, net GND
