File: Thermocouple board Kicad/Thermocouple board/Thermocouple board.kicad_sch (KiCad schematic)
At the start: 8 parts, among them J1 Conn_01x06_Pin, U1 LTC2984CLX-PBF

Commit message: Add files via upload
Parts:
- added J2: Conn_01x02_Pin, Connector_PinHeader_2.54mm:PinHeader_1x02_P2.54mm_Vertical, symbol Connector:Conn_01x02_Pin
- C1, C13, C14, C15, C2, C3: footprint cap:CAPC17595_95N_KEM -> cap:CAP_GRM155R61A106ME11_MUR_0402
- J1: footprint Connector_PinHeader_2.54mm:PinHeader_1x06_P2.54mm_Horizontal -> Connector_PinHeader_2.54mm:PinHeader_1x06_P2.54mm_Vertical
- U1: footprint Processor:LTC2984 -> LTC2984:LQFP-48_LX_LIT
Connections:
- net +3.3V: now also J2.2 (Pin_2)
- net GND: now also J2.1 (Pin_1)
Changed lines of the file:
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@@
 	)
 	(junction
+		(at 104.14 74.93)
+		(diameter 0)
+		(color 0 0 0 0)
+	)
+	(junction
+		(at 123.19 72.39)
+		(diameter 0)
+		(color 0 0 0 0)
+	)
+	(junction
 		(at 120.65 104.14)
 		(diameter 0)
@@
 	(wire
 		(pts
-			(xy 121.92 72.39) (xy 124.46 72.39)
+			(xy 121.92 72.39) (xy 123.19 72.39)
 		)
 		(stroke
@@
 		)
 	)
+	(wire
+		(pts
+			(xy 123.19 72.39) (xy 124.46 72.39)
+		)
+		(stroke
+			(width 0)
+			(type default)
+		)
+	)
 	(bus
 		(pts
@@
 	(wire
 		(pts
+			(xy 123.19 69.85) (xy 123.19 72.39)
+		)
+		(stroke
+			(width 0)
+			(type default)
+		)
+	)
+	(wire
+		(pts
 			(xy 124.46 102.87) (xy 120.65 102.87)
 		)
@@
 	(wire
 		(pts
-			(xy 100.33 74.93) (xy 105.41 74.93)
+			(xy 100.33 74.93) (xy 104.14 74.93)
 		)
 		(stroke
@@
 	(wire
 		(pts
+			(xy 104.14 74.93) (xy 105.41 74.93)
+		)
+		(stroke
+			(width 0)
+			(type default)
+		)
+	)
+	(wire
+		(pts
 			(xy 119.38 104.14) (xy 120.65 104.14)
 		)
@@
 		)
 	)
+	(wire
+		(pts
+			(xy 102.87 69.85) (xy 123.19 69.85)
+		)
+		(stroke
+			(width 0)
+			(type default)
+		)
+	)
 	(bus
 		(pts
@@
 		)
 	)
+	(wire
+		(pts
+			(xy 104.14 72.39) (xy 104.14 74.93)
+		)
+		(stroke
+			(width 0)
+			(type default)
+		)
+	)
 	(bus
 		(pts
@@
 	(wire
 		(pts
+			(xy 102.87 72.39) (xy 104.14 72.39)
+		)
+		(stroke
+			(width 0)
+			(type default)
+		)
+	)
+	(wire
+		(pts
 			(xy 205.74 123.19) (xy 215.9 123.19)
 		)
@@
 			)
 		)
-		(property "Footprint" "cap:CAPC17595_95N_KEM"
+		(property "Footprint" "cap:CAP_GRM155R61A106ME11_MUR_0402"
 			(at 208.28 73.66 0)
 			(effects
@@
 			)
 		)
-		(property "Footprint" "cap:CAPC17595_95N_KEM"
+		(property "Footprint" "cap:CAP_GRM155R61A106ME11_MUR_0402"
 			(at 116.84 104.14 0)
 			(effects
@@
 	)
 	(symbol
+		(lib_id "Connector:Conn_01x02_Pin")
+		(at 97.79 69.85 0)
+		(unit 1)
+		(exclude_from_sim no)
+		(in_bom yes)
+		(on_board yes)
+		(dnp no)
+		(fields_autoplaced yes)
+		(property "Reference" "J2"
+			(at 98.425 64.77 0)
+			(effects
+				(font
+					(size 1.27 1.27)
+				)
+			)
+		)
+		(property "Value" "Conn_01x02_Pin"
+			(at 98.425 67.31 0)
+			(effects
+				(font
+					(size 1.27 1.27)
+				)
+			)
+		)
+		(property "Footprint" "Connector_PinHeader_2.54mm:PinHeader_1x02_P2.54mm_Vertical"
+			(at 97.79 69.85 0)
+			(effects
+				(font
+					(size 1.27 1.27)
+				)
+				(hide yes)
+			)
+		)
+		(property "Datasheet" "~"
+			(at 97.79 69.85 0)
+			(effects
+				(font
+					(size 1.27 1.27)
+				)
+				(hide yes)
+			)
+		)
+		(property "Description" "Generic connector, single row, 01x02, script generated"
+			(at 97.79 69.85 0)
+			(effects
+				(font
+					(size 1.27 1.27)
+				)
+				(hide yes)
+			)
+		)
+		(pin "2"
+		)
+		(pin "1"
+		)
+		(instances
+			(project ""
+				(path "/fa9dc022-1312-44b0-9fb7-b3fdf624cd97"
+					(reference "J2")
+					(unit 1)
+				)
+			)
+		)
+	)
+	(symbol
 		(lib_id "power:GND")
 		(at 38.1 82.55 90)
@@
 			)
 		)
-		(property "Footprint" "Processor:LTC2984"
+		(property "Footprint" "LTC2984:LQFP-48_LX_LIT"
 			(at 124.46 72.39 0)
 			(effects
@@
 			)
 		)
-		(property "Footprint" "Connector_PinHeader_2.54mm:PinHeader_1x06_P2.54mm_Horizontal"
+		(property "Footprint" "Connector_PinHeader_2.54mm:PinHeader_1x06_P2.54mm_Vertical"
 			(at 236.22 95.25 0)
 			(effects
@@
 			)
 		)
-		(property "Footprint" "cap:CAPC17595_95N_KEM"
+		(property "Footprint" "cap:CAP_GRM155R61A106ME11_MUR_0402"
 			(at 210.82 77.47 0)
 			(effects
@@
 			)
 		)
-		(property "Footprint" "cap:CAPC17595_95N_KEM"
+		(property "Footprint" "cap:CAP_GRM155R61A106ME11_MUR_0402"
 			(at 209.55 85.09 0)
 			(effects
@@
 			)
 		)
-		(property "Footprint" "cap:CAPC17595_95N_KEM"
+		(property "Footprint" "cap:CAP_GRM155R61A106ME11_MUR_0402"
 			(at 105.41 80.01 0)
 			(effects
@@
 			)
 		)
-		(property "Footprint" "cap:CAPC17595_95N_KEM"
+		(property "Footprint" "cap:CAP_GRM155R61A106ME11_MUR_0402"
 			(at 118.11 97.79 0)
 			(effects
