File: Thermocouple board Kicad/Thermocouple board/ColdJunction.kicad_sch (KiCad schematic)
At the start: 1 part, among them Q3 2N3904

Commit message: Add files via upload
Parts:
- removed Q3: 2N3904, Package_TO_SOT_THT:TO-92_Inline, symbol Transistor_BJT:2N3904
- added Q1: MMBT3904LT1G, MMBT3904LT1G:SOT95P240X111-3N, symbol BJT:MMBT3904LT1G
Connections:
- net GND: now also Q1.2 (E)
- net VIN: now also Q1.1 (B), Q1.3 (C)
Changed lines of the file:
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@@
 	(wire
 		(pts
-			(xy 99.06 73.66) (xy 99.06 77.47)
+			(xy 97.79 69.85) (xy 97.79 74.93)
 		)
 		(stroke
@@
 	(wire
 		(pts
-			(xy 99.06 87.63) (xy 106.68 87.63)
+			(xy 97.79 90.17) (xy 106.68 90.17)
 		)
 		(stroke
@@
 	(wire
 		(pts
-			(xy 106.68 87.63) (xy 106.68 82.55)
+			(xy 105.41 82.55) (xy 106.68 82.55)
+		)
+		(stroke
+			(width 0)
+			(type default)
+		)
+	)
+	(wire
+		(pts
+			(xy 106.68 82.55) (xy 106.68 90.17)
 		)
 		(stroke
@@
 	(hierarchical_label "GND"
 		(shape input)
-		(at 99.06 73.66 90)
+		(at 97.79 69.85 90)
 		(effects
 			(font
@@
 	)
 	(symbol
-		(lib_id "Transistor_BJT:2N3904")
-		(at 101.6 82.55 180)
+		(lib_id "BJT:MMBT3904LT1G")
+		(at 100.33 82.55 180)
 		(unit 1)
 		(exclude_from_sim no)
@@
 		(dnp no)
 		(fields_autoplaced yes)
-		(property "Reference" "Q3"
+		(property "Reference" "Q1"
 			(at 96.52 81.2799 0)
 			(effects
@@
 			)
 		)
-		(property "Value" "2N3904"
+		(property "Value" "MMBT3904LT1G"
 			(at 96.52 83.8199 0)
 			(effects
@@
 			)
 		)
-		(property "Footprint" "Package_TO_SOT_THT:TO-92_Inline"
-			(at 96.52 80.645 0)
-			(effects
-				(font
-					(size 1.27 1.27)
-					(italic yes)
-				)
-				(justify left)
-				(hide yes)
-			)
-		)
-		(property "Datasheet" "https://www.onsemi.com/pub/Collateral/2N3903-D.PDF"
-			(at 101.6 82.55 0)
+		(property "Footprint" "MMBT3904LT1G:SOT95P240X111-3N"
+			(at 100.33 82.55 0)
 			(effects
 				(font
 					(size 1.27 1.27)
 				)
-				(justify left)
+				(justify bottom)
 				(hide yes)
 			)
 		)
-		(property "Description" "0.2A Ic, 40V Vce, Small Signal NPN Transistor, TO-92"
-			(at 101.6 82.55 0)
+		(property "Datasheet" ""
+			(at 100.33 82.55 0)
 			(effects
 				(font
@@
 			)
 		)
-		(pin "3"
+		(property "Description" ""
+			(at 100.33 82.55 0)
+			(effects
+				(font
+					(size 1.27 1.27)
+				)
+				(hide yes)
+			)
+		)
+		(property "MANUFACTURER" "ON Semiconductor"
+			(at 100.33 82.55 0)
+			(effects
+				(font
+					(size 1.27 1.27)
+				)
+				(justify bottom)
+				(hide yes)
+			)
 		)
 		(pin "2"
+		)
+		(pin "3"
 		)
 		(pin "1"
@@
 			(project ""
 				(path "/fa9dc022-1312-44b0-9fb7-b3fdf624cd97/8afe2570-c552-4a25-a3f0-5c28fbbc8408"
-					(reference "Q3")
+					(reference "Q1")
 					(unit 1)
 				)
