File: Thermocouple board/ColdJunction.kicad_sch (KiCad schematic)
At the start: 1 part, among them Q1 MMBT3904LT1G

Commit message: Add files via upload
Parts:
- Q1: footprint MMBT3904LT1G:SOT95P240X111-3N -> BJT:SOT95P240X111-3N
Changed lines of the file:
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@@
 			)
 		)
-		(property "Footprint" "MMBT3904LT1G:SOT95P240X111-3N"
+		(property "Footprint" "BJT:SOT95P240X111-3N"
 			(at 100.33 82.55 0)
 			(effects
