File: Thermocouple board/Thermocouple board.kicad_pcb (KiCad board)
At the start: 2 copper layers, 54.2 x 87.7 mm, 87 parts, among them J1 Conn_01x06_Pin, J2 Conn_01x02_Pin, Q2 2N3904, Q3 2N3904, U1 LTC2984CLX-PBF

Commit message: Add files via upload
Parts:
- removed J1: Conn_01x06_Pin, Connector_PinHeader_2.54mm:PinHeader_1x06_P2.54mm_Vertical
- removed Q3: 2N3904, BJT:SOT95P240X111-3N
- added J3: Conn_01x07_Socket, Connector_PinHeader_2.54mm:PinHeader_1x07_P2.54mm_Vertical, F.Cu at (131.0, 41.0)
- added Q1: MMBT3904LT1G, BJT:SOT95P240X111-3N, F.Cu at (122.2, 63.1)
- Q2: value 2N3904 -> MMBT3904LT1G
- moved Q2 1.55 mm to (124.1, 50.5)
Connections:
- Q2 pad 1: GND -> /Channel20
- Q2 pad 2: /Channel20 -> GND
Routing:
- net GND: track 74.8 -> 80.5 mm, vias 52 -> 54
- net /Channel20: track 8.89 -> 6.70 mm

Commit message: Add files via upload
Other:
- board text added: "Analog Gnd"
- board text added: "Digital Gnd"
