File: HeatingBoard/Hbridge.kicad_sch (KiCad schematic)
At the start: 26 parts, among them Q1007 ACPL-P347, Q1008 ACPL-P347, Q1009 N-MOSFETT0252, Q1010 N-MOSFETT0252, Q1011 N-MOSFETT0252, Q1012 N-MOSFETT0252, T1004 CON3.81, U1002 NOT(3)TSSOP8

Commit message: Add files via upload
Parts:
- added D2: LED1206, Power:LED-1206, symbol Power-eagle-import:LED1206
- added R2: 1k, Power:R1206, symbol Power-eagle-import:R-EU_R1206
- D1004: COST $0.40 -> $0.23; DIG-PN 160-1643-1-ND -> 160-1643-2-ND
Connections:
- net GND5V: no longer U1002.2 (Y)
- net at D1004.C, Q1011.S, Q1012.D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: now also R2.2
- net at Q1009.S, Q1010.D, R1021.2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: now also D2.C
- new net: D2.A, R2.1
- no-connect marks 2 -> 3
Changed lines of the file:
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@@
+	)
+	(junction
+		(at 167.64 92.71)
+		(diameter 0)
+		(color 0 0 0 0)
 	)
 	(junction
@@
 	)
 	(junction
+		(at 190.5 92.71)
+		(diameter 0)
+		(color 0 0 0 0)
+	)
+	(junction
 		(at 203.2 116.84)
 		(diameter 0)
@@
 	)
 	(no_connect
+		(at 48.26 55.88)
+	)
+	(no_connect
 		(at 99.06 121.92)
 	)
@@
 	(wire
 		(pts
+			(xy 190.5 92.71) (xy 190.5 96.52)
+		)
+		(stroke
+			(width 0.1524)
+			(type solid)
+		)
+	)
+	(wire
+		(pts
 			(xy 96.52 88.9) (xy 99.06 88.9)
 		)
@@
 	(wire
 		(pts
-			(xy 190.5 86.36) (xy 190.5 96.52)
+			(xy 190.5 86.36) (xy 190.5 92.71)
 		)
 		(stroke
@@
 	(wire
 		(pts
+			(xy 189.23 92.71) (xy 190.5 92.71)
+		)
+		(stroke
+			(width 0)
+			(type default)
+		)
+	)
+	(wire
+		(pts
+			(xy 176.53 92.71) (xy 179.07 92.71)
+		)
+		(stroke
+			(width 0)
+			(type default)
+		)
+	)
+	(wire
+		(pts
 			(xy 119.38 93.98) (xy 121.92 93.98)
 		)
@@
 	(wire
 		(pts
+			(xy 167.64 92.71) (xy 168.91 92.71)
+		)
+		(stroke
+			(width 0)
+			(type default)
+		)
+	)
+	(wire
+		(pts
 			(xy 137.16 91.44) (xy 139.7 91.44)
 		)
@@
 	(wire
 		(pts
-			(xy 167.64 86.36) (xy 167.64 96.52)
+			(xy 167.64 86.36) (xy 167.64 92.71)
 		)
 		(stroke
@@
 	(wire
 		(pts
+			(xy 167.64 92.71) (xy 167.64 96.52)
+		)
+		(stroke
+			(width 0.1524)
+			(type solid)
+		)
+	)
+	(wire
+		(pts
 			(xy 132.08 134.62) (xy 121.92 134.62)
 		)
@@
 		(pts
 			(xy 96.52 124.46) (xy 96.52 127)
-		)
-		(stroke
-			(width 0.1524)
-			(type solid)
-		)
-	)
-	(wire
-		(pts
-			(xy 53.34 55.88) (xy 48.26 55.88)
 		)
 		(stroke
@@
 	)
 	(symbol
+		(lib_id "Power-eagle-import:LED1206")
+		(at 173.99 92.71 270)
+		(unit 1)
+		(exclude_from_sim no)
+		(in_bom yes)
+		(on_board yes)
+		(dnp no)
+		(property "Reference" "D2"
+			(at 169.418 89.281 90)
+			(effects
+				(font
+					(size 1.778 1.778)
+				)
+				(justify left bottom)
+			)
+		)
+		(property "Value" "LED1206"
+			(at 169.418 94.615 90)
+			(effects
+				(font
+					(size 1.778 1.778)
+				)
+				(justify left top)
+			)
+		)
+		(property "Footprint" "Power:LED-1206"
+			(at 173.99 92.71 0)
+			(effects
+				(font
+					(size 1.27 1.27)
+				)
+				(hide yes)
+			)
+		)
+		(property "Datasheet" ""
+			(at 173.99 92.71 0)
+			(effects
+				(font
+					(size 1.27 1.27)
+				)
+				(hide yes)
+			)
+		)
+		(property "Description" ""
+			(at 173.99 92.71 0)
+			(effects
+				(font
+					(size 1.27 1.27)
+				)
+				(hide yes)
+			)
+		)
+		(property "COST" "$0.15"
+			(at 173.99 92.71 0)
+			(effects
+				(font
+					(size 1.27 1.27)
+				)
+				(justify left bottom)
+				(hide yes)
+			)
+		)
+		(property "DIG-PN" "  160-1404-2-ND"
+			(at 173.99 92.71 0)
+			(effects
+				(font
+					(size 1.27 1.27)
+				)
+				(justify left bottom)
+				(hide yes)
+			)
+		)
+		(property "MF-PN" " LTST-C150KGKT"
+			(at 173.99 92.71 0)
+			(effects
+				(font
+					(size 1.27 1.27)
+				)
+				(justify left bottom)
+				(hide yes)
+			)
+		)
+		(pin "A"
+		)
+		(pin "C"
+		)
+		(instances
+			(project "HeatingBoard"
+				(path "/f9b4e86f-9747-464e-a8cd-5899416c6d26/cc847f9c-bd14-44b4-b6a2-e8e75a25e39f"
+					(reference "D2")
+					(unit 1)
+				)
+			)
+		)
+	)
+	(symbol
+		(lib_id "Power-eagle-import:R-EU_R1206")
+		(at 184.15 92.71 0)
+		(unit 1)
+		(exclude_from_sim no)
+		(in_bom yes)
+		(on_board yes)
+		(dnp no)
+		(property "Reference" "R2"
+			(at 180.34 91.2114 0)
+			(effects
+				(font
+					(size 1.778 1.5113)
+				)
+				(justify left bottom)
+			)
+		)
+		(property "Value" "1k"
+			(at 180.34 96.012 0)
+			(effects
+				(font
+					(size 1.778 1.5113)
+				)
+				(justify left bottom)
+			)
+		)
+		(property "Footprint" "Power:R1206"
+			(at 184.15 92.71 0)
+			(effects
+				(font
+					(size 1.27 1.27)
+				)
+				(hide yes)
+			)
+		)
+		(property "Datasheet" ""
+			(at 184.15 92.71 0)
+			(effects
+				(font
+					(size 1.27 1.27)
+				)
+				(hide yes)
+			)
+		)
+		(property "Description" ""
+			(at 184.15 92.71 0)
+			(effects
+				(font
+					(size 1.27 1.27)
+				)
+				(hide yes)
+			)
+		)
+		(pin "2"
+		)
+		(pin "1"
+		)
+		(instances
+			(project "HeatingBoard"
+				(path "/f9b4e86f-9747-464e-a8cd-5899416c6d26/cc847f9c-bd14-44b4-b6a2-e8e75a25e39f"
+					(reference "R2")
+					(unit 1)
+				)
+			)
+		)
+	)
+	(symbol
 		(lib_id "Power-eagle-import:R-EU_R1206")
 		(at 144.78 91.44 180)
@@
 			)
 		)
-		(property "COST" "$0.40"
+		(property "COST" "$0.23"
 			(at 182.88 86.36 0)
 			(effects
@@
 			)
 		)
-		(property "DIG-PN" "160-1643-1-ND"
+		(property "DIG-PN" "160-1643-2-ND"
 			(at 182.88 86.36 0)
 			(effects

Commit message: Add files via upload
Fix H-bridge Resistor Value
Parts:
- R1017: value 25R -> 154R
Changed lines of the file:
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@@
 			)
 		)
-		(property "Value" "25R"
+		(property "Value" "154R"
 			(at 148.59 88.138 0)
 			(effects
