File: HeatingBoard/HeatingBoard.kicad_pcb (KiCad board)
At the start: 4 copper layers, 66 parts, among them J1 PJ-080BH, J2 Conn_01x02_Socket, Q1001 ACPL-P347, Q1002 ACPL-P347, Q1003 ACPL-P347, Q1004 N-MOSFETT0252, Q1005 N-MOSFETT0252, Q1006 N-MOSFETT0252, Q1007 ACPL-P347, Q1008 ACPL-P347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

Commit message: Add files via upload
Parts:
- added D2: LED1206, Power:LED-1206, F.Cu at (53.7, 83.8)
- added R2: 1k, Power:R1206, F.Cu at (67.5, 99.6)
- moved R1018 35.6 mm to (54.1, 125.7), turned to 0 degrees
- moved T1004 30.9 mm to (53.7, 91.6), turned to 90 degrees
- moved R1020 30.6 mm to (54.1, 123.5), turned to 180 degrees
- moved D1004 28.4 mm to (53.7, 85.5), turned to 0 degrees
- moved Q1011 20.4 mm to (70.3, 111.2)
- moved Q1010 19.8 mm to (53.7, 114.0), turned to 0 degrees
- moved Q1009 18.4 mm to (61.7, 121.0), turned to 180 degrees
- moved Q1012 16.9 mm to (62.5, 104.4), turned to 180 degrees
- moved R1024 16.8 mm to (73.8, 102.4), turned to 180 degrees
- moved R1017 14.1 mm to (63.0, 112.2), turned to 180 degrees
- moved R1023 11.8 mm to (64.7, 90.5), turned to -90 degrees
- moved C1001 10.9 mm to (112.9, 75.7)
- moved Q1003 10.9 mm to (106.4, 71.3)
- moved C1003 10.8 mm to (132.4, 76.2)
- moved Q1002 10.8 mm to (126.2, 71.8)
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Connections:
- U1002 pad 2: GND5V -> unconnected-(U1002C-Y-Pad2)
Routing:
- net /Hbridge/12VFuse: track 80.9 -> 175.2 mm, vias 10 -> 15
- net Net-(Q1008-Pad5): track 29.8 -> 94.7 mm, vias 0 -> 3
- net Net-(D1004-PadC): track 77.1 -> 30.7 mm, vias 2 -> 0
- net Net-(D2-PadA): track 0.00 -> 23.4 mm
- net Net-(D1004-PadA): track 2.88 -> 23.2 mm, vias 0 -> 2
- net Net-(D2-PadC): track 23.1 -> 41.7 mm
- net GND12V: track 37.3 -> 49.7 mm, vias 20 -> 40
- net Net-(Q1007-Pad5): track 29.8 -> 41.4 mm, vias 0 -> 3
- net Net-(Q1003-Pad5): track 8.71 -> 19.6 mm
- net Net-(Q1002-Pad5): track 8.59 -> 19.4 mm
- net Net-(Q1001-Pad5): track 8.80 -> 19.3 mm
- net Net-(U1001A-Y): track 19.1 -> 9.09 mm
- net Net-(U1001B-Y): track 12.8 -> 3.07 mm
- net Net-(U1001C-Y): track 23.9 -> 16.4 mm
- net GND5V: track 12.9 -> 9.97 mm, vias 7 -> 6
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Other:
- board text added: "+"
- board text added: "+ to -"
- board text added: "-"
- board text added: "- to +"
- board text added: "5V"
- board text added: "Fuse"
- board text added: "GND"
- board text added: "H1"
- board text added: "H2"
- board text added: "H3"
- board text added: "Hbridge1"
- board text added: "Hbridge2"
- board text added: "Inverter"
- board text added: "Min Voltage 11V Max Voltage 13V Norminal 12V at 10A"
- board text added: "On"
- board text added: "Optocoupler"

Commit message: Add files via upload
Other:
- board outline added: 122.4 x 80.8 mm
Changed lines of the file:
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@@
 		(embedded_fonts no)
+	)
+	(gr_rect
+		(start 48.23 46.43)
+		(end 170.59 127.21)
+		(stroke
+			(width 0.1)
+			(type solid)
+		)
+		(fill no)
+		(layer "Edge.Cuts")
 	)
 	(gr_text "On\n"

Commit message: Add files via upload
Fix H-bridge Resistor Value
Parts:
- R1017: value 25R -> 154R
Changed lines of the file:
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@@
 			)
 		)
-		(property "Value" "25R"
+		(property "Value" "154R"
 			(at -1.27 2.54 0)
 			(layer "F.Fab")
